Commit message: Alexis fixed the URDF of boxy by replacing left/right arm.

File: cds_control_nodes/test_data/boxy_fixed_torso_description.urdf (robot description, URDF)
Before this commit: robot boxy_description, 18 links, 17 joints
Links:
- removed link calib_left_arm_base_link
- removed link left_arm_1_link
- removed link left_arm_2_link
- removed link left_arm_3_link
- removed link left_arm_4_link
- removed link left_arm_5_link
- removed link left_arm_6_link
- removed link left_arm_7_link
- added link calib_right_arm_base_link, mass 2.0; collision mesh filename=package://rosie_description/meshes/arm/convex/arm_base_conv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; visual mesh filename=package://rosie_description/meshes/arm/arm_base.stl
- added link right_arm_1_link, mass 2.0; collision mesh filename=package://rosie_description/meshes/arm/convex/arm_segment_a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; visual mesh filename=package://rosie_description/meshes/arm/arm_segment_a.stl
- added link right_arm_2_link, mass 2.0; collision mesh filename=package://rosie_description/meshes/arm/convex/arm_segment_b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; visual mesh filename=package://rosie_description/meshes/arm/arm_segment_b.stl
- added link right_arm_3_link, mass 2.0; collision mesh filename=package://rosie_description/meshes/arm/convex/arm_segment_a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; visual mesh filename=package://rosie_description/meshes/arm/arm_segment_a.stl
- added link right_arm_4_link, mass 2.0; collision mesh filename=package://rosie_description/meshes/arm/convex/arm_segment_b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; visual mesh filename=package://rosie_description/meshes/arm/arm_segment_b.stl
- added link right_arm_5_link, mass 2.0; collision mesh filename=package://rosie_description/meshes/arm/convex/arm_segment_l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; visual mesh filename=package://rosie_description/meshes/arm/arm_segment_last.stl
- added link right_arm_6_link, mass 2.0; collision mesh filename=package://rosie_description/meshes/arm/convex/arm_wrist_con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; visual mesh filename=package://rosie_description/meshes/arm/arm_wrist.stl
- added link right_arm_7_link, mass 2.0; collision mesh filename=package://rosie_description/meshes/arm/convex/arm_flanche_c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; visual mesh filename=package://rosie_description/meshes/arm/arm_flanche.stl
- added link right_arm_flange_link, mass 0.5
- added link triangle_front_center, mass 0.1
Joints:
- removed joint base_link_left_arm_base_joint
- removed joint left_arm_0_joint
- removed joint left_arm_1_joint
- removed joint left_arm_2_joint
- removed joint left_arm_3_joint
- removed joint left_arm_4_joint
- removed joint left_arm_5_joint
- removed joint left_arm_6_joint
- added joint base_link_right_arm_base_joint: type fixed, parent base_link, child calib_right_arm_base_link, origin xyz=0.222335 -0.339149 0.949265 rpy=0.6948481 0.867517 5.5630228
- added joint right_arm_0_joint: type revolute, parent calib_right_arm_base_link, child right_arm_1_link, origin xyz=0 0 0.11 rpy=0 0 0, axis 0 0 1, limit lower=-2.96705972839 upper=2.96705972839 effort=204 velocity=1.91986217719
- added joint right_arm_1_joint: type revolute, parent right_arm_1_link, child right_arm_2_link, origin xyz=0 0 0.20 rpy=0 0 0, axis 0 -1 0, limit lower=-2.09439510239 upper=2.09439510239 effort=306 velocity=1.91986217719
- added joint right_arm_2_joint: type revolute, parent right_arm_2_link, child right_arm_3_link, origin xyz=0 0 0.20 rpy=0 0 0, axis 0 0 1, limit lower=-2.96705972839 upper=2.96705972839 effort=204 velocity=2.26892802759
- added joint right_arm_3_joint: type revolute, parent right_arm_3_link, child right_arm_4_link, origin xyz=0 0 0.20 rpy=0 0 0, axis 0 1 0, limit lower=-2.09439510239 upper=2.09439510239 effort=306 velocity=2.26892802759
- added joint right_arm_4_joint: type revolute, parent right_arm_4_link, child right_arm_5_link, origin xyz=0 0 0.20 rpy=0 0 0, axis 0 0 1, limit lower=-2.96705972839 upper=2.96705972839 effort=204 velocity=2.26892802759
- added joint right_arm_5_joint: type revolute, parent right_arm_5_link, child right_arm_6_link, origin xyz=0 0 0.19 rpy=0 0 0, axis 0 -1 0, limit lower=-2.09439510239 upper=2.09439510239 effort=306 velocity=3.14159265359
- added joint right_arm_6_joint: type revolute, parent right_arm_6_link, child right_arm_7_link, origin xyz=0 0 0 rpy=0 0 0, axis 0 0 1, limit lower=-2.96705972839 upper=2.96705972839 effort=204 velocity=3.14159265359
- added joint right_arm_flange_joint: type fixed, parent right_arm_7_link, child right_arm_flange_link, origin xyz=0 0 0.078 rpy=0 0 0
- added joint triangle_frame_joint: type fixed, parent base_link, child triangle_front_center, origin xyz=0.3625 -0.265 0.85 rpy=0 0 0
